Commit message: Update orca_4fingers_gripper.urdf

File: urdf/orca_4fingers_gripper.urdf (robot description, URDF)
Before this commit: robot orca_4fingers_gripper, 3 links, 2 joints
Joints:
- removed joint roll_jiont1
- removed joint roll_jiont2
- added joint roll_joint1: type revolute, parent base_link, child roll_link1, origin xyz=0.035999 0 -0.087997 rpy=0 0 0, axis 0 -1 0, limit lower=-0.33 upper=0.244 effort=10 velocity=0.1
- added joint roll_joint2: type revolute, parent base_link, child roll_link2, origin xyz=-0.035999 0 -0.087997 rpy=0 0 0, axis 0 -1 0, limit lower=-0.244 upper=0.33 effort=10 velocity=0.1, mimic joint=roll_jiont1 multiplier=-1.0 offset=0
